Commit message: add camera to my_robot

File: my_robot/urdf/robot.urdf.xacro (robot description, xacro)
@@ -4,4 +4,5 @@
     <xacro:arg name="gps_enabled" default="true" />
     <xacro:arg name="imu_enabled" default="true" />
+    <xacro:arg name="camera_enabled" default="true" />
     <xacro:arg name="tf_odom_enabled" default="true" />
     <!-- Include -->
@@ -10,4 +11,5 @@
     <xacro:include filename="$(find my_robot)/urdf/accessories/gps.xacro" />
     <xacro:include filename="$(find my_robot)/urdf/accessories/imu.xacro" />
+    <xacro:include filename="$(find my_robot)/urdf/accessories/usb_camera.xacro" />
     <!-- Body of robot, with plates, standoffs and Create -->
     <xacro:body tf_odom_enabled="$(arg tf_odom_enabled)"/>
@@ -19,5 +21,5 @@
             <child link="laser_link"/>
         </joint>
-        <xacro:rplidar prefix="laser"/>
+        <xacro:rplidar />
     </xacro:if>
     <!-- Attach the GPS -->
@@ -39,3 +41,12 @@
         <xacro:imu />
     </xacro:if>
+    <!-- Attach the Camera -->
+    <xacro:if value="$(arg camera_enabled)">
+        <joint name="camera_joint" type="fixed">
+            <origin xyz="0.15 0 0.1" rpy="0 0 0" />
+            <parent link="base_link"/>
+            <child link="camera_link"/>
+        </joint>
+        <xacro:usb_camera />
+    </xacro:if>
 </robot>

Commit message: my_fsm use /nav_setup to get waypoint

File: my_robot/urdf/robot.urdf.xacro (robot description, xacro)
@@ -44,5 +44,5 @@
     <xacro:if value="$(arg camera_enabled)">
         <joint name="camera_joint" type="fixed">
-            <origin xyz="0.15 0 0.1" rpy="0 0 0" />
+            <origin xyz="0.12 0 0.1" rpy="0 0 0" />
             <parent link="base_link"/>
             <child link="camera_link"/>
