Commit message: change world physics

File: my_robot/urdf/body/body.urdf.xacro (robot description, xacro)
@@ -28,4 +28,9 @@
             <!-- warning: KDL does not support a root link with an inertia. -->
             <!-- <xacro:cylinder_inertial_matrix m="${base_mass}" r="${base_link_radius}" h="${base_link_length}" /> -->
+            <inertial>
+                <mass value="5.0"/>
+                <origin xyz="0 0 0" rpy="0 0 0" />
+                <inertia ixx="1" ixy="0" ixz="0" iyy="1" iyz="0" izz="1"/>
+            </inertial>
         </link>
         <gazebo reference="base_link">

File: my_robot/urdf/body/wheel.urdf.xacro (robot description, xacro)
@@ -24,4 +24,9 @@
             <mu1>5.0</mu1>
             <mu2>5.0</mu2>
+            <kp>10000.0</kp>
+            <kd>10.0</kd>
+            <minDepth>0.0</minDepth>
+            <maxVel>5</maxVel>
+            <fdir1>0 0 0</fdir1>
         </gazebo>
         <joint name="wheel_${lr}_joint" type="continuous">
